File: Hardware/Czujnik_pogody_i_bezpieczenstwa_do_uzytku_domowego.kicad_pcb (KiCad board)
At the start: 4 copper layers, 83 parts, among them IC1 AT25EU0041A-MAHN-T-FLASH, IC2 AP2114HA-3.3TRG1, IC3 MCP73831-2ATI_MC-Battery_char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, IC4 PAM2423AECADJR, J1 MQ-7, J2 USB_C_Receptacle_USB2.0_16P, J4 MQ-2, J5 Wykrywacz_płomieni, J6 Conn_Coaxial-IPX4, Q1 NMOS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

Commit message: Projekt ukończony
Parts:
- removed U1: SMS-202F-Pokrywa EMI, SamacSys:SMS202F
- added 3,3V: TestPoint, TestPoint:TestPoint_THTPad_D1.0mm_Drill0.5mm, F.Cu at (120.6, 123.1)
- added 5V: TestPoint, TestPoint:TestPoint_THTPad_D1.0mm_Drill0.5mm, F.Cu at (153.1, 121.3)
- added BAT+: TestPoint, TestPoint:TestPoint_THTPad_D1.0mm_Drill0.5mm, F.Cu at (177.5, 96.5)
- added BAT-: TestPoint, TestPoint:TestPoint_THTPad_D1.0mm_Drill0.5mm, F.Cu at (145.7, 98.8)
- added C23: 220n, Capacitor_SMD:C_0603_1608Metric, F.Cu at (137.5, 112.9)
- added R21: 1M, Resistor_SMD:R_0805_2012Metric, F.Cu at (141.0, 116.6)
- added R22: 1M, Resistor_SMD:R_0805_2012Metric, F.Cu at (138.0, 116.3)
- moved H1 147.8 mm to (148.1, 101.1)
- moved Q1 146.2 mm to (152.7, 105.8), turned to 0 degrees
- moved C16 138.6 mm to (151.2, 100.9), turned to -90 degrees
- moved U2 136.8 mm to (154.2, 100.9), turned to 180 degrees
- moved R15 133.9 mm to (152.2, 98.1), turned to 180 degrees
- moved R16 133.6 mm to (158.8, 101.8), turned to 0 degrees
- moved Q3 133.0 mm to (160.4, 105.8), turned to 180 degrees
- moved J4 115.5 mm to (174.2, 130.6), turned to -90 degrees
- moved C11 105.7 mm to (164.6, 123.2), turned to -90 degrees
- moved C7 103.1 mm to (166.3, 125.8), turned to 0 degrees
- moved R4 102.3 mm to (140.2, 100.5), turned to -90 degrees
- moved R1 97.7 mm to (170.2, 126.1), turned to 0 degrees
- moved IC4 97.2 mm to (169.8, 121.4), turned to -90 degrees
- moved J2 96.9 mm to (133.8, 97.4)
- moved U4 95.5 mm to (133.2, 109.4), turned to 90 degrees
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Connections:
- net Net-(Q1-D) renamed PMT
- D3 pad 2: Power_USB -> Net-(D3-A)
- IC3 pad 5: Net-(IC3-STAT) -> Net-(D3-K)
- R7 pad 1: Net-(IC3-STAT) -> Net-(D3-A)
- R7 pad 2: Net-(D3-K) -> Power_USB
- U6 pad 10: MQ-2_AOUT -> MQ-7_AOUT
- U6 pad 12: SCL -> SDA
- U6 pad 13: SDA -> SCL
- U6 pad 4: unconnected-(U6-XTAL_32K_P/ADC1_CH0-Pad4) -> Battery_watch
- U6 pad 9: MQ-7_AOUT -> MQ-2_AOUT
Routing:
- net MQ-7_AOUT: track 1.05 -> 62.7 mm, vias 1 -> 2
- net BAT+: track 0.00 -> 47.6 mm, vias 0 -> 5
- net 5V_out: track 0.00 -> 46.1 mm, vias 16 -> 8
- net Wykrywacz_plomieni_out: track 1.42 -> 46.2 mm
- net Net-(D1-K): track 1.18 -> 44.9 mm, vias 1 -> 2
- net 3.3V: track 39.5 -> 82.0 mm, vias 12 -> 15
- net MQ-2_AOUT: track 1.47 -> 43.7 mm, vias 1 -> 2
- net SDA: track 8.58 -> 31.6 mm, vias 1 -> 2
- net SCL: track 4.70 -> 27.6 mm, vias 1 -> 2
- net Battery_watch: track 0.00 -> 20.6 mm, vias 0 -> 2
- net USB_D-: track 0.00 -> 18.3 mm
- net USB_D+: track 0.00 -> 17.0 mm
- net Power_USB: track 13.8 -> 30.6 mm, vias 0 -> 18
- net Net-(J4-Pin_1): track 0.00 -> 16.4 mm, vias 0 -> 2
- net Boost_inductor_out: track 15.1 -> 0.59 mm
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- added copper zone on F.Cu, net 3.3V
- added copper zone on F.Cu, net 5V_out
- added copper zone on F.Cu, net BAT+
- added copper zone on In2.Cu, net BAT+
- added copper zone on F.Cu, net BAT-
- added copper zone on F.Cu, net Boost_inductor_out
- added copper zone on B.Cu, net GND
- added copper zone on In2.Cu, net GND
- added copper zone on F.Cu, net Net-(IC4-EN)
- added copper zone on In2.Cu, net Net-(IC4-EN)
- added copper zone on F.Cu, net PMT
- added copper zone on F.Cu, net Power_USB
- added copper zone on In2.Cu, net Power_USB
Other:
- board outline added: 78 x 40 mm
- board text added: "AHT"
- board text added: "BMP"
- board text added: "Boot"
- board text added: "MQ-2"
- board text added: "MQ-7"
- board text added: "Reset"
