File: Hardware/Czujnik_pogody_i_bezpieczenstwa_do_uzytku_domowego.kicad_sch (KiCad schematic)
At the start: 0 parts

Commit message: Update po dużej ilości pracy
Schemat raczej już skończony.
Parts:
- added C1, C2: C, Capacitor_SMD:C_0603_1608Metric, symbol Device:C
- added C10, C17, C21, C22, C9: 10u, Capacitor_SMD:C_0603_1608Metric, symbol Device:C
- added C11: 1uF, Capacitor_SMD:C_0603_1608Metric, symbol Device:C
- added C12, C13, C15, C16, C18, C19, C26, C27: 100n, Capacitor_SMD:C_0603_1608Metric, symbol Device:C
- added C14, C20: 1u, Capacitor_SMD:C_0603_1608Metric, symbol Device:C
- added C24, C25: 4.7u, Capacitor_SMD:C_0603_1608Metric, symbol Device:C
- added C3, C4: 12p, Capacitor_SMD:C_0603_1608Metric, symbol Device:C
- added C30, C6: 470u, Capacitor_THT:CP_Radial_D10.0mm_P5.00mm, symbol Device:C_Polarized
- added C5: 2.2n, Capacitor_SMD:C_0603_1608Metric, symbol Device:C
- added C7: 47p, Capacitor_SMD:C_0603_1608Metric, symbol Device:C
- added C8: 10n, Capacitor_SMD:C_0603_1608Metric, symbol Device:C
- added D1: Send_LED, LED_SMD:LED_0603_1608Metric, symbol Device:LED
- added D2: Power_LED, LED_SMD:LED_0603_1608Metric, symbol Device:LED
- added D3: Charging_LED, LED_SMD:LED_0603_1608Metric, symbol Device:LED
- added D4, D5: SL82-3G, Diode_SMD:D_SMC, symbol Diode:SS34
- added D6: SMAJ6.0A, Diode_SMD:D_SMA, symbol Diode:SMAJ5.0A
- added H1: Bat-, MountingHole:MountingHole_2.2mm_M2_DIN965_Pad_TopBottom, symbol Mechanical:MountingHole_Pad
- added H2: Bat+, MountingHole:MountingHole_2.2mm_M2_DIN965_Pad_TopBottom, symbol Mechanical:MountingHole_Pad
- added H5, H6, H7, H8: MountingHole_Pad, MountingHole:MountingHole_2.2mm_M2_DIN965_Pad, symbol Mechanical:MountingHole_Pad
- added IC1: AT25EU0041A-MAHN-T-FLASH, SON50P300X200X60-9N-D, symbol SamacSys:AT25EU0041A-MAHN-T
- added IC2: AP2114HA-3.3TRG1, SOT230P700X180-4N, symbol SamacSys_Parts:AP2114HA-3.3TRG1
- added IC3: MCP73831-2ATI_MC-Battery_charge_IC, SON50P300X200X100-9N-D, symbol SamacSys:MCP73831-2ATI_MC
- added IC4: PAM2423AECADJR, PAM2421AECADJR, symbol SamacSys_Parts:PAM2421AECADJR
- added J1: MQ-7, Connector_PinSocket_2.54mm:PinSocket_1x04_P2.54mm_Vertical, symbol Connector:Conn_01x04_Socket
- added J2: USB_C_Receptacle_USB2.0_16P, Connector_USB:USB_C_Receptacle_GCT_USB4105-xx-A_16P_TopMnt_Horizontal, symbol Connector:USB_C_Receptacle_USB2.0_16P
- added J4: MQ-2, Connector_PinSocket_2.54mm:PinSocket_1x04_P2.54mm_Vertical, symbol Connector:Conn_01x04_Socket
- added J5: Wykrywacz_płomieni, Connector_PinSocket_2.54mm:PinSocket_1x03_P2.54mm_Vertical, symbol Connector:Conn_01x03_Socket
- added J6: Conn_Coaxial-IPX4, SamacSys:IPX4, symbol Connector:Conn_Coaxial
- added L1: L, Inductor_SMD:L_0603_1608Metric, symbol Device:L
- added L2: 2.2u, Moje_inductory:DR127, symbol Device:L
- added L3: 2n2, Inductor_SMD:L_0603_1608Metric, symbol Device:L
- added Q1, Q3: NMOS, Package_SO:SOP-8_3.76x4.96mm_P1.27mm, symbol Simulation_SPICE:NMOS
- added Q2: AO3401A, Package_TO_SOT_SMD:SOT-23, symbol Transistor_FET:AO3401A
- added R1: 51k, Resistor_SMD:R_0805_2012Metric, symbol Device:R
- added R10, R3, R4: 5.1k, Resistor_SMD:R_0805_2012Metric, symbol Device:R
- added R11: 100k, Resistor_SMD:R_0805_2012Metric, symbol Device:R
- added R12, R5, R6, R8: 10k, Resistor_SMD:R_0805_2012Metric, symbol Device:R
- added R13, R14, R7: 1k, Resistor_SMD:R_0805_2012Metric, symbol Device:R
- added R15: 330, Resistor_SMD:R_0805_2012Metric, symbol Device:R
- added R16: 2.7k, Resistor_SMD:R_0805_2012Metric, symbol Device:R
- added R17, R18, R19, R20: 20k, Resistor_SMD:R_0805_2012Metric, symbol Device:R
- added R2: 15k, Resistor_SMD:R_0805_2012Metric, symbol Device:R
- added R9: 2k, Resistor_SMD:R_0805_2012Metric, symbol Device:R
- added S1: Reset_switch, RKC2SJM170SMTRLFS, symbol SamacSys:RKC2SJM170SMTRLFS
- added S2: Boot_switch, RKC2SJM170SMTRLFS, symbol SamacSys:RKC2SJM170SMTRLFS
- added TP1: TestPoint, symbol Connector:TestPoint
- added U1: SMS-202F-Pokrywa EMI, SMS202F, symbol SamacSys:SMS-202F
- added U2: AP9101CK6, Package_TO_SOT_SMD:SOT-23-6, symbol Battery_Management:AP9101CK6
- added U3: AHT20, AHT20, symbol SamacSys:AHT20
- added U4: SRV05-4, Package_TO_SOT_SMD:SOT-23-6, symbol Power_Protection:SRV05-4
- added U5: BMP280, Package_LGA:Bosch_LGA-8_2x2.5mm_P0.65mm_ClockwisePinNumbering, symbol Sensor_Pressure:BMP280
- added U6: ESP32-C3, Package_DFN_QFN:QFN-32-1EP_5x5mm_P0.5mm_EP3.45x3.45mm, symbol PCM_Espressif:ESP32-C3
- added Y2: Crystal_GND24, Crystal:Crystal_SMD_3225-4Pin_3.2x2.5mm, symbol Device:Crystal_GND24
Connections:
- new net: R8.2, S2.1 (COM_1), S2.2 (COM_2), U6.15 (GPIO9/BOOT)
- new net: C14.1, R5.2, S1.3 (NO_1), S1.4 (NO_2), U6.7 (CHIP_EN)
- new net: C11.1, C22.1, C6.1, IC4.2 (VIN), IC4.3 (EN), L2.1, Q2.2 (S)
- new net: C1.1, L1.2, U6.1 (LNA_IN)
- new net: R12.2, U6.14 (GPIO8)
- new net: D1.1 (K), U6.16 (GPIO10)
- new net: IC1.7 (~{HOLD_(IO3)}), U6.19 (SPIHD/GPIO12)
- new net: C18.1, L3.2, U6.2 (VDD3P3), U6.3 (VDD3P3)
- new net: IC1.3 (~{WP_(IO2_ACC)}), U6.20 (SPIWP/GPIO13)
- new net: IC1.1 (~{CS}), U6.21 (SPICS0/GPIO14)
- new net: IC1.6 (SCK), U6.22 (SPICLK/GPIO15)
- new net: IC1.5 (SI_(IO0)), U6.23 (SPID/GPIO16)
- new net: IC1.2 (SO_(IO1)), U6.24 (SPIQ/GPIO17)
- new net: C3.1, U6.29 (XTAL_N), Y2.1
- new net: C4.1, U6.30 (XTAL_P), Y2.3
- new net: R6.2, U6.6 (GPIO2/ADC1_CH2)
- new net: J1.1 (Pin_1), R17.2
- new net: Q1.1 (D), Q3.1 (D)
- new net: Q3.2 (G), U2.3 (CO)
- new net: C5.1, R1.2
- new net: C7.1, IC4.4 (COMP), R1.1
- new net: J2.B5 (CC2), R3.1
- new net: D1.2 (A), R13.1
- new net: C2.2, J6.1 (In), L1.1
- new net: Q2.1 (G), R11.1
- new net: Q1.2 (G), U2.1 (DO)
- new net: J4.1 (Pin_1), R19.2
- new net: D2.2 (A), R14.1
- new net: IC4.6 (FB), R10.1, R2.2
- new net: D3.1 (K), R7.2
- new net: R16.1, U2.2 (VM)
- new net: J2.A5 (CC1), R4.1
- new net: C16.1, R15.2, U2.5 (VDD)
- new net: IC3.5 (STAT), R7.1
- new net: IC3.8 (PROG), R9.1
- new net: C8.1, IC4.7 (SS)
- new net 3.3V: C12.1, C13.1, C15.2, C19.1, C20.1, C21.1, C26.1, C27.1, C9.1, IC1.8 (VCC), IC2.3 (VOUT), J5.1 (Pin_1), L3.1, R12.1, R13.2, R14.2, R5.1, R6.1, R8.1, U3.2 (VDD), U5.2 (CSB), U5.6 (VDDIO), U5.8 (VDD), U6.11 (VDD3P3_RTC), U6.17 (VDD3P3_CPU), U6.31 (VDDA), U6.32 (VDDA)
- new net 5V_out: C10.2, C17.1, C30.1, D4.1 (K), D5.1 (K), IC2.1 (VIN), J1.4 (Pin_4), J4.4 (Pin_4), R2.1
- new net BAT+: C24.1, H2.1, IC3.3 (VBAT_1), IC3.4 (VBAT_2), Q2.3 (D), R15.1
- new net BAT-: C16.2, H1.1, Q1.3 (S), U2.6 (VSS)
- new net Boost_inductor_out: D4.2 (A), IC4.8 (SW), L2.2
- new net GND: C1.2, C10.1, C11.2, C12.2, C13.2, C14.2, C15.1, C17.2, C18.2, C19.2, C2.1, C20.2, C21.2, C22.2, C24.2, C25.2, C26.2, C27.2, C3.2, C30.2, C4.2, C5.2, C6.2, C7.2, C8.2, C9.2, D2.1 (K), D6.2 (A2), H5.1, H6.1, H7.1, H8.1, IC1.4 (GND), IC1.9 (EP), IC2.2 (GND_1), IC2.4 (GND_2), IC3.6 (VSS), IC3.9 (EP), IC4.1 (PGND), IC4.5 (AGND), IC4.9 (EP), J1.3 (Pin_3), J2.A1 (GND), J2.A12 (GND), J2.B1 (GND), J2.B12 (GND), J2.S1 (SHIELD), J4.3 (Pin_3), J5.2 (Pin_2), J6.2 (Ext), Q3.3 (S), R10.2, R16.2, R18.1, R20.1, R3.2, R4.2, R9.2, S1.1 (COM_1), S1.2 (COM_2), S2.3 (NO_1), S2.4 (NO_2), U1.1, U1.10, U1.11, U1.12, U1.2, U1.3, U1.4, U1.5, U1.6, U1.7, U1.8, U1.9, U3.5 (GND), U4.2 (VN), U5.1 (GND), U5.7 (GND), U6.33 (GND), Y2.2 (G), Y2.4 (G)
- new net MQ-2_AOUT: R19.1, R20.2, U6.10 (MTDI/GPIO5/ADC2_CH0)
- new net MQ-2_DOUT: J4.2 (Pin_2)
- new net MQ-7_AOUT: R17.1, R18.2, U6.9 (MTMS/GPIO4/ADC1_CH4)
- new net MQ-7_DOUT: J1.2 (Pin_2)
- new net Power_USB: C25.1, D3.2 (A), D5.2 (A), D6.1 (A1), IC3.1 (VDD_1), IC3.2 (VDD_2), J2.A4 (VBUS), J2.A9 (VBUS), J2.B4 (VBUS), J2.B9 (VBUS), R11.2, U4.5 (VP)
- new net SCL: U3.3 (SCL), U5.4 (SCK), U6.12 (MTCK/GPIO6)
- new net SDA: U3.4 (SDA), U5.5 (SDO), U6.13 (MTDO/GPIO7)
- new net USB_D+: J2.A6 (D+), J2.B6 (D+), U4.1 (IO1), U4.6 (IO4), U6.26 (GPIO19/USB_D+)
- new net USB_D-: J2.A7 (D-), J2.B7 (D-), U4.3 (IO2), U4.4 (IO3), U6.25 (GPIO18/USB_D-)
- new net Wykrywacz_plomieni_out: J5.3 (Pin_3), U6.8 (GPIO3/ADC1_CH3)
- no-connect marks 0 -> 1
Other:
- note added: "Boost konwerter dla uzyskania 5V 3A"
- note added: "Układ ochrony baterii"
- note added: "Wkręty na śruby"

Commit message: Projekt ukończony
Parts:
- removed U1: SMS-202F-Pokrywa EMI, SMS202F, symbol SamacSys:SMS-202F
- added C23: 220n, Capacitor_SMD:C_0603_1608Metric, symbol Device:C
- added R21, R22: 1M, Resistor_SMD:R_0805_2012Metric, symbol Device:R
- added TP2, TP3, TP4: TestPoint, TestPoint:TestPoint_THTPad_D1.0mm_Drill0.5mm, symbol Connector:TestPoint
- TP1: footprint (none) -> TestPoint:TestPoint_THTPad_D1.0mm_Drill0.5mm
Connections:
- net 3.3V: now also TP1.1
- net 5V_out: now also TP2.1
- net BAT+: now also R21.2, TP3.1
- net BAT-: now also TP4.1
- net GND: now also C23.2, R22.2
- net MQ-2_AOUT: now also U6.9 (MTMS/GPIO4/ADC1_CH4); no longer U6.10 (MTDI/GPIO5/ADC2_CH0)
- net MQ-7_AOUT: now also U6.10 (MTDI/GPIO5/ADC2_CH0); no longer U6.9 (MTMS/GPIO4/ADC1_CH4)
- net Power_USB: now also R7.2; no longer D3.2 (A)
- net SCL: now also U6.13 (MTDO/GPIO7); no longer U6.12 (MTCK/GPIO6)
- net SDA: now also U6.12 (MTCK/GPIO6); no longer U6.13 (MTDO/GPIO7)
- net Battery_watch: now reaches U6.4 (XTAL_32K_P/ADC1_CH0)
- net Battery_watch: now also C23.1, R21.1, R22.1
- net PMT: now reaches Q1.1 (D), Q3.1 (D)
- net at D3.1 (K): now also IC3.5 (STAT); no longer R7.2
- net at R7.1: now also D3.2 (A); no longer IC3.5 (STAT)
- no-connect marks 1 -> 0
Other:
- note added: "Upewnij się że ogarnąłeś AGND"
- moved on the sheet: D3, R7
